Commit message: Diff drive controller added

File: rb1_ros2_description/xacro/rb1_ros2_base.urdf.xacro (robot description, xacro)
@@ -86,3 +86,33 @@
 	<!-- Gazebo ros2 control plugins -->
 	<!-- <xacro:ros2_control/> -->
+    <ros2_control name="diff_drive" type="system">
+        <hardware>
+            <plugin>gazebo_ros2_control/GazeboSystem</plugin>
+        </hardware>
+        <joint name="robot_left_wheel_joint">
+            <command_interface name="velocity">
+            <param name="min">-1</param>
+            <param name="max">1</param>
+            </command_interface>
+            <state_interface name="position"/>
+            <state_interface name="velocity"/>
+            <state_interface name="effort"/>
+        </joint>
+        <joint name="robot_right_wheel_joint">
+            <command_interface name="velocity">
+            <param name="min">-1</param>
+            <param name="max">1</param>
+            </command_interface>
+            <state_interface name="position"/>
+            <state_interface name="velocity"/>
+            <state_interface name="effort"/>
+        </joint>
+    </ros2_control>
+    <gazebo>
+        <plugin filename="libgazebo_ros2_control.so" name="gazebo_ros2_control">
+            <robot_sim_type>gazebo_ros2_control/DefaultRobotHWSim</robot_sim_type>
+            <parameters>$(find rb1_ros2_description)/config/rb1_controller.yaml</parameters>
+            <robot_param_node>/robot_state_publisher</robot_param_node>
+        </plugin>
+    </gazebo>
 </robot>

Commit message: Differential drive controller added to RB1

File: rb1_ros2_description/xacro/rb1_ros2_base.urdf.xacro (robot description, xacro)
@@ -18,4 +18,7 @@
 	<!-- Import Elevator -->
 	<xacro:include filename="$(find rb1_ros2_description)/urdf/elevator/elevator.urdf.xacro"/>
+	<!-- Import ROS2 Control -->
+	<!-- <xacro:include filename="$(find rb1_ros2_description)/xacro/rb1.ros2_control.xacro"/>
+	<xacro:include filename="$(find rb1_ros2_description)/xacro/rb1.gazebo.xacro"/> -->
 	<!-- ***************** -->
 	<!-- Global parameters -->
@@ -41,6 +44,8 @@
 	<xacro:property name="elevator_z" value="0.213" />
 	<xacro:arg name="prefix" default="robot_"/>
+    <xacro:property name="robot_name" value="rb1_robot"/>
 	<xacro:arg name="ros_planar_move_plugin" default="false"/>
 	<xacro:arg name="gpu" default="false"/>
+    <xacro:arg name="use_sim" default="true" />
 	<!-- *************** -->
 	<!-- Robots Elements -->
@@ -85,5 +90,6 @@
 	</xacro:sensor_orbbec_astra>
 	<!-- Gazebo ros2 control plugins -->
-	<!-- <xacro:ros2_control/> -->
+	<!-- <xacro:rb1_ros2_control prefix="$(arg prefix)" name="rb1" use_sim="$(arg use_sim)" />
+	<xacro:rb1_gazebo prefix="$(arg prefix)" />  -->
     <ros2_control name="diff_drive" type="system">
         <hardware>
@@ -108,10 +114,17 @@
             <state_interface name="effort"/>
         </joint>
+        <!-- <joint name="robot_elevator_platform_joint">
+            <command_interface name="effort">
+            <param name="min">0</param>
+            <param name="max">10</param>
+            </command_interface>
+            <state_interface name="position"/>
+            <state_interface name="velocity"/>
+            <state_interface name="effort"/>
+        </joint> -->
     </ros2_control>
     <gazebo>
         <plugin filename="libgazebo_ros2_control.so" name="gazebo_ros2_control">
-            <robot_sim_type>gazebo_ros2_control/DefaultRobotHWSim</robot_sim_type>
             <parameters>$(find rb1_ros2_description)/config/rb1_controller.yaml</parameters>
-            <robot_param_node>/robot_state_publisher</robot_param_node>
         </plugin>
     </gazebo>

Commit message: xacro modified to add elevator joint

File: rb1_ros2_description/xacro/rb1_ros2_base.urdf.xacro (robot description, xacro)
@@ -114,5 +114,5 @@
             <state_interface name="effort"/>
         </joint>
-        <!-- <joint name="robot_elevator_platform_joint">
+        <joint name="robot_elevator_platform_joint">
             <command_interface name="effort">
             <param name="min">0</param>
@@ -122,5 +122,5 @@
             <state_interface name="velocity"/>
             <state_interface name="effort"/>
-        </joint> -->
+        </joint>
     </ros2_control>
     <gazebo>
